Commit message: set the motion of the robot

File: ufactory-xarm-uf850/uf850_description/urdf/uf850.urdf (robot description, URDF)
Before this commit: robot uf850, 7 links, 6 joints
Joints:
- joint base_to_link1: axis (none) -> 0 0 1; limit (none) -> lower=0.0 upper=0.3 effort=10 velocity=0.5; type fixed -> continuous
- joint link1_to_link2: axis (none) -> 0 1 0; limit (none) -> lower=-1.57 upper=1.57 effort=10.0 velocity=1.0; type fixed -> revolute
- joint link2_to_link3: axis (none) -> 0 0 1; limit (none) -> lower=-4.71 upper=0 effort=10.0 velocity=1.0; type fixed -> revolute
- joint link3_to_link4: axis (none) -> 1 0 0; type fixed -> continuous
- joint link4_to_link5: axis (none) -> 0 1 0; type fixed -> continuous
- joint link5_to_link6: axis (none) -> 0 0 1; type fixed -> continuous
